Commit message: Add URDF mesh example

File: urdf/prarob_manipulator.xacro (robot description, xacro)
@@ -9,6 +9,6 @@
     <axis xyz="0 0 1" />
   </joint>
-  <!-- Link 1 -->
-  <link name="link1">
+  <!-- Link 1 - primitives-->
+  <!--link name="link1">
     <visual>
       <origin xyz="0 0 0.5" rpy="0 0 0"/>
@@ -22,4 +22,22 @@
       <geometry>
         <box size="0.05 0.05 1.0"/>
+      </geometry>
+    </collision>
+  </link-->
+<!-- Link 1 - stl -->
+  <link name="link1">
+    <visual>
+      <origin rpy="0 0 0" xyz="0 0 0"/>
+      <geometry>
+        <mesh filename="package://ros2_prarob/meshes/postolje_seminar_v1.stl" scale="0.01 0.01 0.01"/>
+      </geometry>
+      <material name="">
+        <color rgba="0.054901960784313725 0.054901960784313725 0.06274509803921569 1.0"/>
+      </material>
+    </visual>
+    <collision>
+      <origin rpy="0 0 0" xyz="0 0 0"/>
+      <geometry>
+        <mesh filename="package://ros2_prarob/meshes/postolje_seminar_v1.stl" scale="0.01 0.01 0.01"/>
       </geometry>
     </collision>

Commit message: added urdf v1 with links and joints,

File: urdf/prarob_manipulator.xacro (robot description, xacro)
@@ -1,3 +1,3 @@
-<?xml version="1.0"?>
+<?xml version="1.0" ?>
 <robot xmlns:xacro="http://ros.org/wiki/xacro">
 <xacro:macro name="prarob_manipulator" params="parent *origin">
@@ -9,110 +9,183 @@
     <axis xyz="0 0 1" />
   </joint>
-  <!-- Link 1 - primitives-->
-  <!--link name="link1">
-    <visual>
-      <origin xyz="0 0 0.5" rpy="0 0 0"/>
-      <geometry>
-        <box size="0.05 0.05 1.0"/>
-      </geometry>
-      <color rgba="0 0 0.8 1"/>
-    </visual>
-    <collision>
-      <origin xyz="0 0 0" rpy="0 0 0"/>
-      <geometry>
-        <box size="0.05 0.05 1.0"/>
-      </geometry>
-    </collision>
-  </link-->
-<!-- Link 1 - stl -->
-  <link name="link1">
-    <visual>
-      <origin rpy="0 0 0" xyz="0 0 0"/>
-      <geometry>
-        <mesh filename="package://ros2_prarob/meshes/postolje_seminar_v1.stl" scale="0.01 0.01 0.01"/>
-      </geometry>
-      <material name="">
-        <color rgba="0.054901960784313725 0.054901960784313725 0.06274509803921569 1.0"/>
-      </material>
-    </visual>
-    <collision>
-      <origin rpy="0 0 0" xyz="0 0 0"/>
-      <geometry>
-        <mesh filename="package://ros2_prarob/meshes/postolje_seminar_v1.stl" scale="0.01 0.01 0.01"/>
-      </geometry>
-    </collision>
-  </link>
-  <!-- Joint 1 -->
-  <joint name="joint1" type="revolute">
-    <parent link="link1"/>
-    <child link="link2"/>
-    <origin xyz="0.0 0.0 1.0" rpy="0 0 0"/>
-    <axis xyz="0 0 1"/>
-    <limit velocity="10.0" effort="1" lower="-2.82743338823" upper="2.82743338823" />
-  </joint>
-  <!-- Link 2 -->
-  <link name="link2">
-    <visual>
-      <origin xyz="0 0 0.3" rpy="0 0 0"/>
-      <geometry>
-        <box size="0.05 0.05 0.6"/>
-      </geometry>
-      <color rgba="0 0.8 0.0 1"/>
-    </visual>
-    <collision>
-      <origin xyz="0 0 0.3" rpy="0 0 0"/>
-      <geometry>
-        <box size="0.05 0.05 0.6"/>
-      </geometry>
-    </collision>
-  </link>
-  <!-- Joint 2 -->
-  <joint name="joint2" type="revolute">
-    <parent link="link2"/>
-    <child link="link3"/>
-    <origin xyz="0.0 0.0 0.60" rpy="0 0 0"/>
-    <axis xyz="1 0 0"/>
-    <limit velocity="10.0" effort="1" lower="-2.82743338823" upper="2.82743338823" />
-  </joint>
-  <!-- Link 3 -->
-  <link name="link3">
-    <visual>
-      <origin xyz="0.15 0 0" rpy="0 0 0"/>
-      <geometry>
-        <box size="0.3 0.05 0.05"/>
-      </geometry>
-      <color rgba="0 0 0.8 1"/>
-    </visual>
-    <collision>
-      <origin xyz="0 0 0" rpy="0 0 0"/>
-      <geometry>
-        <box size="0.3 0.05 0.05"/>
-      </geometry>
-    </collision>
-  </link>
-  <!-- Joint 2 -->
-  <joint name="joint3" type="revolute">
-    <parent link="link3"/>
-    <child link="link_tool"/>
-    <origin xyz="0.3 0.0 0.0" rpy="0 0 0"/>
-    <axis xyz="1 0 0"/>
-    <limit velocity="10.0" effort="1" lower="-2.82743338823" upper="2.82743338823" />
-  </joint>
-  <!-- link_tool -->
-  <link name="link_tool">
-    <visual>
-      <origin xyz="0 0 0" rpy="0 0 0"/>
-      <geometry>
-        <box size="0.08 0.08 0.08"/>
-      </geometry>
-      <color rgba="0 0 0.8 1"/>
-    </visual>
-    <collision>
-      <origin xyz="0 0 0" rpy="0 0 0"/>
-      <geometry>
-        <box size="0.08 0.08 0.08"/>
-      </geometry>
-    </collision>
-  </link>
+<xacro:include filename="$(find ros2_prarob)/urdf/materials.xacro" />
+<!-- xacro:include filename="$(find ros2_prarob)/urdf/prarob_manipulator.trans" / -->
+<!-- xacro:include filename="$(find ros2_prarob)/urdf/prarob_manipulator.gazebo" / -->
+<link name="link1">
+  <!-- inertial>
+    <origin xyz="0.0 0.0 0.0" rpy="0 0 0"/>
+    <mass value="0.0"/>
+    <inertia ixx="0.0" iyy="0.0" izz="0.0" ixy="0.0" iyz="0.0" ixz="0.0"/>
+  </inertial -->
+  <visual>
+    <origin xyz="0 0 0" rpy="0 0 0"/>
+    <geometry>
+      <mesh filename="package://ros2_prarob/meshes/Postolje.stl" scale="0.001 0.001 0.001"/>
+    </geometry>
+    <material name="silver"/>
+  </visual>
+  <collision>
+    <origin xyz="0 0 0" rpy="0 0 0"/>
+    <geometry>
+      <mesh filename="package://ros2_prarob/meshes/Postolje.stl" scale="0.001 0.001 0.001"/>
+    </geometry>
+  </collision>
+</link>
+<link name="XL-430-DUMMY_1">
+  <!-- inertial>
+    <origin xyz="0.04552107498052348 -0.008523635973404789 0.04077229889987345" rpy="0 0 0"/>
+    <mass value="0.32236070836601705"/>
+    <inertia ixx="5e-05" iyy="8.6e-05" izz="7.8e-05" ixy="-0.0" iyz="-0.0" ixz="-2e-06"/>
+  </inertial -->
+  <visual>
+    <origin xyz="0.070882 -0.028065 0.042342" rpy="0 0 0"/>
+    <geometry>
+      <mesh filename="package://ros2_prarob/meshes/XL-430-DUMMY.stl" scale="0.001 0.001 0.001"/>
+    </geometry>
+    <material name="silver"/>
+  </visual>
+  <collision>
+    <origin xyz="0.070882 -0.028065 0.042342" rpy="0 0 0"/>
+    <geometry>
+      <mesh filename="package://ros2_prarob/meshes/XL-430-DUMMY.stl" scale="0.001 0.001 0.001"/>
+    </geometry>
+  </collision>
+</link>
+<link name="link2">
+  <!-- inertial>
+    <origin xyz="1.313686505965972e-07 3.799087183557759e-07 0.007236548561630161" rpy="0 0 0"/>
+    <mass value="0.051205577518979827"/>
+    <inertia ixx="5e-06" iyy="1.2e-05" izz="1.4e-05" ixy="-0.0" iyz="-0.0" ixz="0.0"/>
+  </inertial -->
+  <visual>
+    <origin xyz="0.013441 -0.019532 -0.016329" rpy="0 0 0"/>
+    <geometry>
+      <mesh filename="package://ros2_prarob/meshes/Link_90.stl" scale="0.001 0.001 0.001"/>
+    </geometry>
+    <material name="silver"/>
+  </visual>
+  <collision>
+    <origin xyz="0.013441 -0.019532 -0.016329" rpy="0 0 0"/>
+    <geometry>
+      <mesh filename="package://ros2_prarob/meshes/Link_90.stl" scale="0.001 0.001 0.001"/>
+    </geometry>
+  </collision>
+</link>
+<link name="XL-430-DUMMY_2">
+  <!-- inertial>
+    <origin xyz="0.03154239274272504 -0.008541604373071877 0.0007509813313925362" rpy="0 0 0"/>
+    <mass value="0.32236070836601705"/>
+    <inertia ixx="7.8e-05" iyy="8.6e-05" izz="5e-05" ixy="0.0" iyz="0.0" ixz="-2e-06"/>
+  </inertial -->
+  <visual>
+    <origin xyz="0.043882 -0.028065 -0.051658" rpy="0 0 0"/>
+    <geometry>
+      <mesh filename="package://ros2_prarob/meshes/XL-430-DUMMY.stl" scale="0.001 0.001 0.001"/>
+    </geometry>
+    <material name="silver"/>
+  </visual>
+  <collision>
+    <origin xyz="0.043882 -0.028065 -0.051658" rpy="0 0 0"/>
+    <geometry>
+      <mesh filename="package://ros2_prarob/meshes/XL-430-DUMMY.stl" scale="0.001 0.001 0.001"/>
+    </geometry>
+  </collision>
+</link>
+<link name="link3">
+  <!-- inertial>
+    <origin xyz="0.004211318281894754 3.7974480672151034e-07 0.10000003920965964" rpy="0 0 0"/>
+    <mass value="0.13371939999286847"/>
+    <inertia ixx="0.000606" iyy="0.0006" izz="7e-06" ixy="0.0" iyz="0.0" ixz="-0.0"/>
+  </inertial -->
+  <visual>
+    <origin xyz="-0.005559 -0.019532 -0.064329" rpy="0 0 0"/>
+    <geometry>
+      <mesh filename="package://ros2_prarob/meshes/Link_RR.stl" scale="0.001 0.001 0.001"/>
+    </geometry>
+    <material name="silver"/>
+  </visual>
+  <collision>
+    <origin xyz="-0.005559 -0.019532 -0.064329" rpy="0 0 0"/>
+    <geometry>
+      <mesh filename="package://ros2_prarob/meshes/Link_RR.stl" scale="0.001 0.001 0.001"/>
+    </geometry>
+  </collision>
+</link>
+<link name="XL-430-DUMMY_3">
+  <!-- inertial>
+    <origin xyz="-0.017898607257275104 9.363862685157764e-06 0.011920097087554649" rpy="0 0 0"/>
+    <mass value="0.32236070836601705"/>
+    <inertia ixx="7.8e-05" iyy="8.6e-05" izz="5e-05" ixy="-0.0" iyz="0.0" ixz="2e-06"/>
+  </inertial -->
+  <visual>
+    <origin xyz="-0.005559 -0.019532 -0.264329" rpy="0 0 0"/>
+    <geometry>
+      <mesh filename="package://ros2_prarob/meshes/XL-430-DUMMY.stl" scale="0.001 0.001 0.001"/>
+    </geometry>
+    <material name="silver"/>
+  </visual>
+  <collision>
+    <origin xyz="-0.005559 -0.019532 -0.264329" rpy="0 0 0"/>
+    <geometry>
+      <mesh filename="package://ros2_prarob/meshes/XL-430-DUMMY.stl" scale="0.001 0.001 0.001"/>
+    </geometry>
+  </collision>
+</link>
+<link name="link_tool">
+  <!-- inertial>
+    <origin xyz="-0.29957315293648246 -0.026440620091279402 0.05057202391299859" rpy="0 0 0"/>
+    <mass value="0.05021305846733036"/>
+    <inertia ixx="6e-06" iyy="8e-06" izz="8e-06" ixy="0.0" iyz="0.0" ixz="-1e-06"/>
+  </inertial -->
+  <visual>
+    <origin xyz="-0.282888 -0.045973 -0.255797" rpy="0 0 0"/>
+    <geometry>
+      <mesh filename="package://ros2_prarob/meshes/Izvrsni_clan.stl" scale="0.001 0.001 0.001"/>
+    </geometry>
+    <material name="silver"/>
+  </visual>
+  <collision>
+    <origin xyz="-0.282888 -0.045973 -0.255797" rpy="0 0 0"/>
+    <geometry>
+      <mesh filename="package://ros2_prarob/meshes/Izvrsni_clan.stl" scale="0.001 0.001 0.001"/>
+    </geometry>
+  </collision>
+</link>
+<joint name="rigid1" type="fixed">
+  <origin xyz="-0.070882 0.028065 -0.042342" rpy="0 0 0"/>
+  <parent link="link1"/>
+  <child link="XL-430-DUMMY_1"/>
+</joint>
+<joint name="rigid2" type="fixed">
+  <origin xyz="-0.030441 0.008533 0.035329" rpy="0 0 0"/>
+  <parent link="link2"/>
+  <child link="XL-430-DUMMY_2"/>
+</joint>
+<joint name="rigid3" type="fixed">
+  <origin xyz="0.277329 0.026441 -0.008532" rpy="0 0 0"/>
+  <parent link="XL-430-DUMMY_3"/>
+  <child link="link_tool"/>
+</joint>
+<joint name="joint1" type="revolute">
+  <origin xyz="0.057441 -0.008533 0.058671" rpy="0 0 0"/>
+  <parent link="XL-430-DUMMY_1"/>
+  <child link="link2"/>
+  <axis xyz="0.0 0.0 1.0"/>
+  <limit velocity="10.0" effort="1" lower="-2.82743338823" upper="2.82743338823" />
+</joint>
+<joint name="joint2" type="revolute">
+  <origin xyz="0.049441 -0.008533 0.012671" rpy="0 0 0"/>
+  <parent link="XL-430-DUMMY_2"/>
+  <child link="link3"/>
+  <axis xyz="1.0 0.0 0.0"/>
+  <limit velocity="10.0" effort="1" lower="-2.82743338823" upper="2.82743338823" />
+</joint>
+<joint name="joint3" type="revolute">
+  <origin xyz="0.0 0.0 0.2" rpy="0 0 0"/>
+  <parent link="link3"/>
+  <child link="XL-430-DUMMY_3"/>
+  <axis xyz="1.0 0.0 0.0"/>
+  <limit velocity="10.0" effort="1" lower="-2.82743338823" upper="2.82743338823" />
+</joint>
 </xacro:macro>
 </robot>

Commit message: updated launch file to run everything, added direct kinematics publishing, fixed bugs

File: urdf/prarob_manipulator.xacro (robot description, xacro)
@@ -147,5 +147,6 @@
 </joint>
 <joint name="joint3" type="revolute">
-   <origin xyz="-2.0000000298e-01 6.2172489379e-17 -6.2172489379e-17" rpy="3.141593 0.0 1.570796"/>
+  <origin xyz="-2.0000000298e-01 6.2172489379e-17 -6.2172489379e-17" rpy="3.141593 0.0 0.0"/>
+  <!-- origin xyz="-2.0000000298e-01 6.2172489379e-17 -6.2172489379e-17" rpy="3.141593 0.0 1.570796"/-->
   <parent link="link3"/>
   <child link="XL-430-DUMMY_3"/>

Commit message: pathplanning fixed, urdf needs fixing

File: urdf/prarob_manipulator.xacro (robot description, xacro)
@@ -74,5 +74,6 @@
 <link name="link3">
   <visual>
-     <origin xyz="-1.0000000149e-01 0.0000000000e+00 -4.1000000000e-03" rpy="0.0 0.0 0.0"/>
+     <origin xyz="-1.0000000149e-01 0.0000000000e+00 -4.1000000000e-03" rpy="3.141593 0.0 3.141593"/>
+     <!--origin xyz="-1.0000000149e-01 0.0000000000e+00 -4.1000000000e-03" rpy="0.0 0.0 0.0"/-->
     <geometry>
       <mesh filename="package://ros2_prarob/meshes/Link_RR.stl" scale="0.001 0.001 0.001"/>
@@ -140,5 +141,5 @@
 </joint>
 <joint name="joint2" type="revolute">
-  <origin xyz="4.4408920985e-18 -4.4408920985e-18 2.0900000000e-02" rpy="-3.141593 0.0 -1.570796"/>
+  <origin xyz="4.4408920985e-18 -4.4408920985e-18 2.0900000000e-02" rpy="0.0 0.0 1.570796"/>
   <parent link="XL-430-DUMMY_2"/>
   <child link="link3"/>

Commit message: working direct kinematics, inverse toDo

File: urdf/prarob_manipulator.xacro (robot description, xacro)
@@ -74,5 +74,5 @@
 <link name="link3">
   <visual>
-     <origin xyz="-1.0000000149e-01 0.0000000000e+00 -4.1000000000e-03" rpy="3.141593 0.0 3.141593"/>
+     <origin xyz="-1.0000000149e-01 0.0000000000e+00 -4.1000000000e-03" rpy="0.0 0.0 0.0"/>
      <!--origin xyz="-1.0000000149e-01 0.0000000000e+00 -4.1000000000e-03" rpy="0.0 0.0 0.0"/-->
     <geometry>
@@ -141,16 +141,16 @@
 </joint>
 <joint name="joint2" type="revolute">
-  <origin xyz="4.4408920985e-18 -4.4408920985e-18 2.0900000000e-02" rpy="0.0 0.0 1.570796"/>
+  <origin xyz="4.4408920985e-18 -4.4408920985e-18 2.0900000000e-02" rpy="-3.141593 0.0 -1.570796"/>
   <parent link="XL-430-DUMMY_2"/>
   <child link="link3"/>
-  <axis xyz="0.0 0.0 1.0"/>
+  <axis xyz="0.0 0.0 -1.0"/>
   <limit velocity="10.0" effort="1" lower="-2.82743338823" upper="2.82743338823" />
 </joint>
 <joint name="joint3" type="revolute">
-  <origin xyz="-2.0000000298e-01 6.2172489379e-17 -6.2172489379e-17" rpy="3.141593 0.0 0.0"/>
+  <origin xyz="-2.0000000298e-01 6.2172489379e-17 -6.2172489379e-17" rpy="3.141593 0.0 1.570796"/>
   <!-- origin xyz="-2.0000000298e-01 6.2172489379e-17 -6.2172489379e-17" rpy="3.141593 0.0 1.570796"/-->
   <parent link="link3"/>
   <child link="XL-430-DUMMY_3"/>
-  <axis xyz="0.0 0.0 1.0"/>
+  <axis xyz="0.0 0.0 -1.0"/>
   <limit velocity="10.0" effort="1" lower="-2.82743338823" upper="2.82743338823" />
 </joint>
